File: digital clock.kicad_sch (KiCad schematic)
At the start: 156 parts, among them Q1 BC557, Q10 BC547, Q11 BC547, Q12 BC557, Q13 BC557, Q14 BC557, Q2 BC557, Q3 BC557, Q7 BC557, Q8 BC547, Q9 BC547

Commit message: display board
Parts:
- added J1: Conn_01x14_Socket, Connector_Molex:Molex_SL_171971-0014_1x14_P2.54mm_Vertical, symbol Connector:Conn_01x14_Socket
- added Q4: BC547, Package_TO_SOT_THT:TO-92_Inline, symbol Transistor_BJT:BC547
- added R35: 10k, Resistor_THT:R_Axial_DIN0207_L6.3mm_D2.5mm_P10.16mm_Horizontal, symbol Device:R_US
- added R36: 1k, Resistor_THT:R_Axial_DIN0207_L6.3mm_D2.5mm_P10.16mm_Horizontal, symbol Device:R_US
- added R37: 33, Resistor_THT:R_Axial_DIN0207_L6.3mm_D2.5mm_P10.16mm_Horizontal, symbol Device:R_US
- D100, D101, D102, D103, D104, D105, D106, D107, D108, D109, D110, D111, D112, D113, D114, D115, D116, D117, D118, D119, D120, D121, D122, D123, D124, D125, D126, D127, D128, D129, D130, D131, D132, D133, D134, D135, D136, D137, D138, D139, D140, D141, D142, D143, D144, D23, D25, D27, D32, D33, D34, D35, D36, D37, D38, D39, D40, D41, D42, D43, D44, D45, D46, D47, D48, D49, D50, D51, D52, D53, D54, D55, D56, D57, D58, D59, D60, D61, D62, D63, D64, D65, D66, D67, D68, D69, D70, D71, D72, D73, D74, D75, D76, D77, D78, D79, D80, D81, D82, D83, D84, D85, D86, D87, D88, D89, D90, D91, D92, D93, D94, D95, D96, D97, D98, D99: footprint LED_THT:LED_D3.0mm -> LED_THT:LED_D5.0mm
- R10, R16, R18, R21, R26, R29, R30, R33, R34, R8: value 1k -> 10k
- R11, R12, R13, R15, R17, R19, R22, R23, R27, R9: value 10k -> 1k
Connections:
- net GND: now also J1.14 (Pin_14), Q4.3 (E)
- net Led A: now also J1.6 (Pin_6)
- net Led B: now also J1.7 (Pin_7)
- net Led C: now also J1.8 (Pin_8)
- net Led D: now also J1.9 (Pin_9)
- net Led E: now also J1.10 (Pin_10)
- net Led F: now also J1.11 (Pin_11)
- net Led G: now also J1.12 (Pin_12)
- net Vcc: now also D100.1 (K), D101.1 (K), D102.1 (K), D103.1 (K), D104.1 (K), D105.1 (K), D106.1 (K), D107.1 (K), D108.1 (K), D109.1 (K), D110.1 (K), D111.1 (K), D112.1 (K), D117.1 (K), D118.1 (K), D119.1 (K), D120.1 (K), D121.1 (K), D122.1 (K), D123.1 (K), D124.1 (K), D125.1 (K), D126.1 (K), D127.1 (K), D128.1 (K), D129.1 (K), D130.1 (K), D131.1 (K), D132.1 (K), D133.1 (K), D134.1 (K), D135.1 (K), D136.1 (K), D137.1 (K), D138.1 (K), D139.1 (K), D140.1 (K), D141.1 (K), D142.1 (K), D143.1 (K), D144.1 (K), D23.1 (K), D25.1 (K), D27.1 (K), D32.1 (K), D33.1 (K), D34.1 (K), D35.1 (K), D36.1 (K), D37.1 (K), D38.1 (K), D39.1 (K), D40.1 (K), D41.1 (K), D42.1 (K), D43.1 (K), D44.1 (K), D45.1 (K), D46.1 (K), D47.1 (K), D48.1 (K), D49.1 (K), D50.1 (K), D51.1 (K), D52.1 (K), D53.1 (K), D54.1 (K), D55.1 (K), D56.1 (K), D57.1 (K), D58.1 (K), D59.1 (K), D60.1 (K), D61.1 (K), D62.1 (K), D63.1 (K), D64.1 (K), D65.1 (K), D66.1 (K), D67.1 (K), D68.1 (K), D69.1 (K), D70.1 (K), D71.1 (K), D72.1 (K), D73.1 (K), D74.1 (K), D75.1 (K), D76.1 (K), D77.1 (K), D78.1 (K), D79.1 (K), D80.1 (K), D81.1 (K), D82.1 (K), D83.1 (K), D84.1 (K), D85.1 (K), D86.1 (K), D87.1 (K), D88.1 (K), D89.1 (K), D90.1 (K), D91.1 (K), D92.1 (K), D93.1 (K), D94.1 (K), D95.1 (K), D96.1 (K), D97.1 (K), D98.1 (K), D99.1 (K), Q10.1 (C), Q11.1 (C), Q8.1 (C), Q9.1 (C), R10.2, R21.2, R26.2, J1.13 (Pin_13), Q4.1 (C), R35.1, R37.2; no longer R10.1, R21.1, R22.1, R23.1, R24.1, R26.1, R27.1
- net at D115.1 (K): now also D113.1 (K), D114.1 (K), D116.1 (K), R37.1
- net at D115.2 (A): now also D113.2 (A), D114.2 (A), D116.2 (A)
- net at Q10.2 (B): now also R24.2; no longer R25.2
- new net: Q4.2 (B), R36.2
- new net SQW: J1.5 (Pin_5), R35.2, R36.1
- new net digit 1: J1.1 (Pin_1), R10.1, R22.1
- new net digit 2: J1.2 (Pin_2), R21.1, R23.1
- new net digit 3: J1.3 (Pin_3), R24.1, R25.2
- new net digit 4: J1.4 (Pin_4), R26.1, R27.1
Other:
- sheet MCU ports: added Led_A, Led_B, Led_C, Led_D, Led_E, Led_F, Led_G, SQW, Vcc, digit 1, digit 2, digit 3, digit 4; removed none
- sheet power circuit ports: added +12v, Vcc; removed none
- moved on the sheet: D113, D114, D115, D116, R10, R21, R22, R24, R25, R26
