File: digital clock.kicad_pcb (KiCad board)
At the start: 2 copper layers, 214 x 150 mm, 166 parts, among them Q1 BC557, Q10 BC547, Q11 BC547, Q12 BC557, Q13 BC557, Q14 BC557, Q2 BC557, Q3 BC557, Q7 BC557, Q8 BC547, Q9 BC547, SW1 SW_Push, SW2 SW_Push, SW3 SW_Wuerth_450301014042, U1 LM337_TO220, U2 ATmega328-P, U3 DS3231M

Commit message: transistor correction and LEDs arrangement
Parts:
- added R28: R_US, Resistor_THT:R_Axial_DIN0309_L9.0mm_D3.2mm_P12.70mm_Horizontal, F.Cu at (169.3, 127.0)
- added R29: R_US, Resistor_THT:R_Axial_DIN0207_L6.3mm_D2.5mm_P10.16mm_Horizontal, F.Cu at (169.3, 131.4)
- added R30: R_US, Resistor_THT:R_Axial_DIN0207_L6.3mm_D2.5mm_P10.16mm_Horizontal, F.Cu at (169.3, 135.4)
- added R31: R_US, Resistor_THT:R_Axial_DIN0204_L3.6mm_D1.6mm_P7.62mm_Horizontal, F.Cu at (169.2, 139.1)
- added R32: R_US, Resistor_THT:R_Axial_DIN0204_L3.6mm_D1.6mm_P7.62mm_Horizontal, F.Cu at (169.2, 142.2)
- added R33: R_US, Resistor_THT:R_Axial_DIN0204_L3.6mm_D1.6mm_P7.62mm_Horizontal, F.Cu at (169.2, 145.3)
- added R34: R_US, Resistor_THT:R_Axial_DIN0204_L3.6mm_D1.6mm_P7.62mm_Horizontal, F.Cu at (169.2, 148.5)
- moved D120 155.6 mm to (251.9, 26.6)
- moved D121 155.6 mm to (251.9, 32.1)
- moved D122 155.6 mm to (251.9, 37.7)
- moved D123 155.6 mm to (251.9, 43.2)
- moved D124 155.6 mm to (251.9, 48.8)
- moved D125 155.6 mm to (251.9, 54.4)
- moved D126 155.6 mm to (251.9, 59.9)
- moved D127 155.6 mm to (251.9, 65.5)
- moved D128 155.6 mm to (251.9, 71.0)
- moved D129 155.6 mm to (251.9, 76.5)
- moved D130 155.6 mm to (251.9, 82.1)
- moved D131 155.6 mm to (251.9, 87.7)
- moved D132 155.6 mm to (251.9, 93.2)
- moved D133 155.6 mm to (257.8, 26.6)
- moved D134 155.6 mm to (257.8, 32.1)
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Connections:
- D100 pad 2: GND -> /G
- D101 pad 2: GND -> /D
- D102 pad 2: GND -> /A
- D103 pad 2: GND -> /G
- D104 pad 2: GND -> /D
- D105 pad 2: GND -> /B
- D106 pad 2: GND -> /B
- D107 pad 2: GND -> /B
- D108 pad 2: GND -> /B
- D109 pad 2: GND -> /C
- D110 pad 2: GND -> /C
- D111 pad 2: GND -> /C
- D112 pad 2: GND -> /C
- D117 pad 2: GND -> /F
- D118 pad 2: GND -> /F
- D119 pad 2: GND -> /F
- D120 pad 2: GND -> /F
- D121 pad 2: GND -> /E
- D122 pad 2: GND -> /E
- D123 pad 2: GND -> /E
- D124 pad 2: GND -> /E
- D125 pad 2: GND -> /A
- D126 pad 2: GND -> /G
- D127 pad 2: GND -> /D
- D128 pad 2: GND -> /A
- D129 pad 2: GND -> /G
- D130 pad 2: GND -> /D
- D131 pad 2: GND -> /A
- D132 pad 2: GND -> /G
- D133 pad 2: GND -> /D
- D134 pad 2: GND -> /A
- D135 pad 2: GND -> /G
- D136 pad 2: GND -> /D
- D137 pad 2: GND -> /B
- D138 pad 2: GND -> /B
- D139 pad 2: GND -> /B
- D140 pad 2: GND -> /B
- D141 pad 2: GND -> /C
- D142 pad 2: GND -> /C
- D143 pad 2: GND -> /C
- D144 pad 2: GND -> /C
- D23 pad 2: GND -> /F
- D25 pad 2: GND -> /F
- D27 pad 2: GND -> /F
- D32 pad 2: GND -> /F
- D33 pad 2: GND -> /F
- D34 pad 2: GND -> /F
- D35 pad 2: GND -> /F
- D36 pad 2: GND -> /F
- D37 pad 2: GND -> /E
- D38 pad 2: GND -> /E
- D39 pad 2: GND -> /E
- D40 pad 2: GND -> /E
- D41 pad 2: GND -> /A
- D42 pad 2: GND -> /G
- D43 pad 2: GND -> /D
- D44 pad 2: GND -> /A
- D45 pad 2: GND -> /G
- D46 pad 2: GND -> /D
- D47 pad 2: GND -> /A
- D48 pad 2: GND -> /G
- D49 pad 2: GND -> /D
- D50 pad 2: GND -> /A
- D51 pad 2: GND -> /G
- D52 pad 2: GND -> /D
- D53 pad 2: GND -> /E
- D54 pad 2: GND -> /B
- D55 pad 2: GND -> /E
- D56 pad 2: GND -> /B
- D57 pad 2: GND -> /E
- D58 pad 2: GND -> /B
- D59 pad 2: GND -> /E
- D60 pad 2: GND -> /B
- D61 pad 2: GND -> /C
- D62 pad 2: GND -> /C
- D63 pad 2: GND -> /C
- D64 pad 2: GND -> /C
- D65 pad 2: GND -> /A
- D66 pad 2: GND -> /G
- D67 pad 2: GND -> /D
- D68 pad 2: GND -> /A
- D69 pad 2: GND -> /G
- D70 pad 2: GND -> /D
- D71 pad 2: GND -> /A
- D72 pad 2: GND -> /G
- D73 pad 2: GND -> /D
- D74 pad 2: GND -> /A
- D75 pad 2: GND -> /G
- D76 pad 2: GND -> /D
- D77 pad 2: GND -> /B
- D78 pad 2: GND -> /B
- D79 pad 2: GND -> /B
- D80 pad 2: GND -> /B
- D81 pad 2: GND -> /C
- D82 pad 2: GND -> /C
- D83 pad 2: GND -> /C
- D84 pad 2: GND -> /C
- D85 pad 2: GND -> /F
- D86 pad 2: GND -> /F
- D87 pad 2: GND -> /F
- D88 pad 2: GND -> /F
- D89 pad 2: GND -> /E
- D90 pad 2: GND -> /E
- D91 pad 2: GND -> /E
- D92 pad 2: GND -> /E
- D93 pad 2: GND -> /A
- D94 pad 2: GND -> /G
- D95 pad 2: GND -> /D
- D96 pad 2: GND -> /A
- D97 pad 2: GND -> /G
- D98 pad 2: GND -> /D
- D99 pad 2: GND -> /A
- R11 pad 1: GND -> /GPIO
- R12 pad 2: GND -> /GPIO
- R13 pad 1: GND -> /GPIO
- R14 pad 1: GND -> /C
- R15 pad 1: GND -> /GPIO
- R16 pad 1: GND -> /GPIO
- R16 pad 2: Net-(Q12-C) -> /Vcc
- R17 pad 1: GND -> /GPIO
- R18 pad 1: GND -> /GPIO
- R18 pad 2: Net-(Q13-C) -> /Vcc
- R19 pad 1: GND -> /GPIO
- R20 pad 1: GND -> /G
- R6 pad 1: GND -> /B
- R7 pad 1: GND -> /D
- R8 pad 1: GND -> /GPIO
- R8 pad 2: Net-(Q1-C) -> /Vcc
- R9 pad 1: GND -> /GPIO

Commit message: Changes to be committed:
Parts:
- R1, R10, R11, R12, R13, R14, R15, R16, R17, R18, R19, R2, R20, R21, R22, R23, R24, R25, R26, R27, R3, R31, R32, R33, R34, R4, R5, R6, R7, R8, R9: footprint Resistor_THT:R_Axial_DIN0204_L3.6mm_D1.6mm_P7.62mm_Horizontal -> Resistor_THT:R_Axial_DIN0207_L6.3mm_D2.5mm_P10.16mm_Horizontal
- R28: footprint Resistor_THT:R_Axial_DIN0309_L9.0mm_D3.2mm_P12.70mm_Horizontal -> Resistor_THT:R_Axial_DIN0207_L6.3mm_D2.5mm_P10.16mm_Horizontal
- moved D113 136.0 mm to (112.2, 35.5)
- moved D114 135.9 mm to (112.2, 41.5)
- moved D115 134.9 mm to (111.7, 58.0)
- moved D116 134.9 mm to (111.7, 64.0)
- moved R23 115.9 mm to (186.9, 90.9)
- moved R22 115.9 mm to (186.9, 87.8)
- moved R24 115.9 mm to (186.9, 94.0)
- moved R25 115.9 mm to (186.9, 97.2)
- moved R26 115.9 mm to (186.9, 100.3)
- moved R27 115.9 mm to (186.9, 103.5)
- moved D117 102.6 mm to (160.2, 25.9)
- moved D118 102.3 mm to (160.2, 31.9)
- moved D119 102.1 mm to (160.2, 37.9)
- moved D131 99.4 mm to (178.2, 20.9)
- moved D124 94.6 mm to (160.2, 71.9)
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
Commit message: value addition & led arrangement
Parts:
- R10, R16, R18, R2, R21, R24, R26, R29, R3, R30, R33, R34, R4, R5, R8: value R_US -> 1k
- R11, R12, R13, R15, R17, R19, R22, R23, R25, R27, R9: value R_US -> 10k
- R14, R20, R28, R31, R32, R6, R7: value R_US -> 33
- moved Q8 227.4 mm to (36.4, 89.3), turned to 90 degrees
- moved R10 202.3 mm to (47.5, 94.0), turned to 90 degrees
- moved R21 195.0 mm to (85.0, 93.1), turned to 90 degrees
- moved Q9 187.9 mm to (75.5, 89.3), turned to 90 degrees
- moved R22 143.5 mm to (43.5, 83.9), turned to -90 degrees
- moved Q10 132.8 mm to (130.4, 89.3), turned to 90 degrees
- moved R23 106.4 mm to (80.5, 93.1), turned to 90 degrees
- moved R28 99.7 mm to (198.3, 21.0)
- moved Q11 96.0 mm to (167.0, 89.0), turned to 90 degrees
- moved R31 86.9 mm to (198.4, 63.0)
- moved R29 82.8 mm to (208.6, 38.5), turned to 180 degrees
- moved R32 82.3 mm to (198.3, 52.5)
- moved R20 74.1 mm to (198.4, 73.5)
- moved R30 65.9 mm to (208.5, 49.0), turned to 180 degrees
- moved Q3 64.0 mm to (216.6, 32.7), turned to -90 degrees
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Connections:
- R11 pad 1: /GPIO -> /Led D
- R12 pad 2: /GPIO -> /Led A
- R13 pad 1: /GPIO -> /Led C
- R15 pad 1: /GPIO -> /Led E
- R16 pad 1: /GPIO -> /Led E
- R17 pad 1: /GPIO -> /Led F
- R18 pad 1: /GPIO -> /Led F
- R19 pad 1: /GPIO -> /Led G
- R29 pad 2: /GPIO -> /Led B
- R30 pad 2: /GPIO -> /Led C
- R33 pad 1: /GPIO -> /Led G
- R34 pad 1: /GPIO -> /Led D
- R8 pad 1: /GPIO -> /Led A
- R9 pad 1: /GPIO -> /Led B
- U2 pad 1: unconnected-(U2-~{RESET}/PC6-Pad1) -> /MCU/RST
- U2 pad 11: unconnected-(U2-PD5-Pad11) -> /MCU/Led D
- U2 pad 12: unconnected-(U2-PD6-Pad12) -> /MCU/Led E
- U2 pad 14: unconnected-(U2-PB0-Pad14) -> /MCU/Led G
- U2 pad 4: unconnected-(U2-PD2-Pad4) -> /MCU/Led A
- U2 pad 5: unconnected-(U2-PD3-Pad5) -> /MCU/Led B
- U2 pad 6: unconnected-(U2-PD4-Pad6) -> /MCU/Led C
- U3 pad 4: unconnected-(U3-~{RST}-Pad4) -> /MCU/RST

Commit message: display board
Parts:
- added J1: Conn_01x14_Socket, Connector_Molex:Molex_SL_171971-0014_1x14_P2.54mm_Vertical, F.Cu at (290.5, 157.7)
- added J1: Conn_01x14_Socket, Connector_Molex:Molex_SL_171971-0014_1x14_P2.54mm_Vertical, F.Cu at (288.3, 244.0)
- added J2: Conn_01x06_Socket, Connector_PinHeader_2.54mm:PinHeader_1x06_P2.54mm_Vertical, F.Cu at (234.3, 257.0)
- added Q4: BC547, Package_TO_SOT_THT:TO-92_Inline, F.Cu at (137.4, 118.3)
- added R35: 10k, Resistor_THT:R_Axial_DIN0207_L6.3mm_D2.5mm_P10.16mm_Horizontal, F.Cu at (143.8, 123.5)
- added R36: 1k, Resistor_THT:R_Axial_DIN0207_L6.3mm_D2.5mm_P10.16mm_Horizontal, F.Cu at (153.7, 117.0)
- added R37: 33, Resistor_THT:R_Axial_DIN0207_L6.3mm_D2.5mm_P10.16mm_Horizontal, F.Cu at (152.1, 106.0)
- D100, D101, D102, D103, D104, D105, D106, D107, D108, D109, D110, D111, D112, D113, D114, D115, D116, D117, D118, D119, D120, D121, D122, D123, D124, D125, D126, D127, D128, D129, D130, D131, D132, D133, D134, D135, D136, D137, D138, D139, D140, D141, D142, D143, D144, D23, D25, D27, D32, D33, D34, D35, D36, D37, D38, D39, D40, D41, D42, D43, D44, D45, D46, D47, D48, D49, D50, D51, D52, D53, D54, D55, D56, D57, D58, D59, D60, D61, D62, D63, D64, D65, D66, D67, D68, D69, D70, D71, D72, D73, D74, D75, D76, D77, D78, D79, D80, D81, D82, D83, D84, D85, D86, D87, D88, D89, D90, D91, D92, D93, D94, D95, D96, D97, D98, D99: footprint LED_THT:LED_D3.0mm -> LED_THT:LED_D5.0mm
- R10, R16, R18, R21, R26, R29, R30, R33, R34, R8: value 1k -> 10k
- R11, R12, R13, R15, R17, R19, R22, R23, R27, R9: value 10k -> 1k
- moved R5 167.8 mm to (239.1, 200.8)
- moved SW1 167.8 mm to (222.6, 222.6)
- moved SW2 167.8 mm to (184.4, 222.8)
- moved SW3 167.8 mm to (205.9, 227.3)
- moved C5 167.8 mm to (217.1, 205.9)
- moved U2 167.8 mm to (182.9, 182.1)
- moved U3 167.8 mm to (222.2, 197.9)
- moved R4 162.8 mm to (245.8, 189.3)
- moved R3 148.4 mm to (231.1, 184.8)
- moved RV1 143.2 mm to (132.5, 245.4), turned to 90 degrees
- moved C3 123.4 mm to (161.0, 224.5), turned to -90 degrees
- moved R1 115.2 mm to (162.0, 249.6), turned to 90 degrees
- moved C4 113.1 mm to (153.5, 224.5), turned to -90 degrees
- moved R2 109.7 mm to (204.2, 180.3)
- moved U1 102.6 mm to (153.5, 241.4), turned to -90 degrees
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Connections:
- net +12V renamed /power circuit/+12v
- C3 pad 1: Net-(U1-VO) -> /Vcc
- C4 pad 1: Net-(U1-VO) -> /Vcc
- C5 pad 1: /MCU/Vcc -> /Vcc
- D100 pad 1: Net-(D100-K) -> /Vcc
- D101 pad 1: Net-(D100-K) -> /Vcc
- D102 pad 1: Net-(D100-K) -> /Vcc
- D103 pad 1: Net-(D100-K) -> /Vcc
- D104 pad 1: Net-(D100-K) -> /Vcc
- D105 pad 1: Net-(D100-K) -> /Vcc
- D106 pad 1: Net-(D100-K) -> /Vcc
- D107 pad 1: Net-(D100-K) -> /Vcc
- D108 pad 1: Net-(D100-K) -> /Vcc
- D109 pad 1: Net-(D100-K) -> /Vcc
- D110 pad 1: Net-(D100-K) -> /Vcc
- D111 pad 1: Net-(D100-K) -> /Vcc
- D112 pad 1: Net-(D100-K) -> /Vcc
- D113 pad 1: unconnected-(D113-K-Pad1) -> Net-(D113-K)
- D113 pad 2: unconnected-(D113-A-Pad2) -> Net-(D113-A)
- D114 pad 1: unconnected-(D114-K-Pad1) -> Net-(D113-K)
- D114 pad 2: unconnected-(D114-A-Pad2) -> Net-(D113-A)
- D115 pad 1: unconnected-(D115-K-Pad1) -> Net-(D113-K)
- D115 pad 2: unconnected-(D115-A-Pad2) -> Net-(D113-A)
- D116 pad 1: unconnected-(D116-K-Pad1) -> Net-(D113-K)
- D116 pad 2: unconnected-(D116-A-Pad2) -> Net-(D113-A)
- D117 pad 1: Net-(D117-K) -> /Vcc
- D118 pad 1: Net-(D117-K) -> /Vcc
- D119 pad 1: Net-(D117-K) -> /Vcc
- D120 pad 1: Net-(D117-K) -> /Vcc
- D121 pad 1: Net-(D117-K) -> /Vcc
- D122 pad 1: Net-(D117-K) -> /Vcc
- D123 pad 1: Net-(D117-K) -> /Vcc
- D124 pad 1: Net-(D117-K) -> /Vcc
- D125 pad 1: Net-(D117-K) -> /Vcc
- D126 pad 1: Net-(D117-K) -> /Vcc
- D127 pad 1: Net-(D117-K) -> /Vcc
- D128 pad 1: Net-(D117-K) -> /Vcc
- D129 pad 1: Net-(D117-K) -> /Vcc
- D130 pad 1: Net-(D117-K) -> /Vcc
- D131 pad 1: Net-(D117-K) -> /Vcc
- D132 pad 1: Net-(D117-K) -> /Vcc
- D133 pad 1: Net-(D117-K) -> /Vcc
- D134 pad 1: Net-(D117-K) -> /Vcc
- D135 pad 1: Net-(D117-K) -> /Vcc
- D136 pad 1: Net-(D117-K) -> /Vcc
- D137 pad 1: Net-(D117-K) -> /Vcc
- D138 pad 1: Net-(D117-K) -> /Vcc
- D139 pad 1: Net-(D117-K) -> /Vcc
- D140 pad 1: Net-(D117-K) -> /Vcc
- D141 pad 1: Net-(D117-K) -> /Vcc
- D142 pad 1: Net-(D117-K) -> /Vcc
- D143 pad 1: Net-(D117-K) -> /Vcc
- D144 pad 1: Net-(D117-K) -> /Vcc
- D23 pad 1: Net-(D23-K) -> /Vcc
- D25 pad 1: Net-(D23-K) -> /Vcc
- D27 pad 1: Net-(D23-K) -> /Vcc
- D32 pad 1: Net-(D23-K) -> /Vcc
- D33 pad 1: Net-(D33-K) -> /Vcc
- D34 pad 1: Net-(D33-K) -> /Vcc
- D35 pad 1: Net-(D33-K) -> /Vcc
- D36 pad 1: Net-(D33-K) -> /Vcc
- D37 pad 1: Net-(D33-K) -> /Vcc
- D38 pad 1: Net-(D33-K) -> /Vcc
- D39 pad 1: Net-(D33-K) -> /Vcc
- D40 pad 1: Net-(D33-K) -> /Vcc
- D41 pad 1: Net-(D33-K) -> /Vcc
- D42 pad 1: Net-(D33-K) -> /Vcc
- D43 pad 1: Net-(D33-K) -> /Vcc
- D44 pad 1: Net-(D33-K) -> /Vcc
- D45 pad 1: Net-(D33-K) -> /Vcc
- D46 pad 1: Net-(D33-K) -> /Vcc
- D47 pad 1: Net-(D33-K) -> /Vcc
- D48 pad 1: Net-(D33-K) -> /Vcc
- D49 pad 1: Net-(D33-K) -> /Vcc
- D50 pad 1: Net-(D33-K) -> /Vcc
- D51 pad 1: Net-(D33-K) -> /Vcc
- D52 pad 1: Net-(D33-K) -> /Vcc
- D53 pad 1: Net-(D23-K) -> /Vcc
- D54 pad 1: Net-(D33-K) -> /Vcc
- D55 pad 1: Net-(D23-K) -> /Vcc
- D56 pad 1: Net-(D33-K) -> /Vcc
- D57 pad 1: Net-(D23-K) -> /Vcc
- D58 pad 1: Net-(D33-K) -> /Vcc
- D59 pad 1: Net-(D23-K) -> /Vcc
- D60 pad 1: Net-(D33-K) -> /Vcc
- D61 pad 1: Net-(D33-K) -> /Vcc
- D62 pad 1: Net-(D33-K) -> /Vcc
- D63 pad 1: Net-(D33-K) -> /Vcc
- D64 pad 1: Net-(D33-K) -> /Vcc
- D65 pad 1: Net-(D23-K) -> /Vcc
- D66 pad 1: Net-(D23-K) -> /Vcc
- D67 pad 1: Net-(D23-K) -> /Vcc
- D68 pad 1: Net-(D23-K) -> /Vcc
- D69 pad 1: Net-(D23-K) -> /Vcc
- D70 pad 1: Net-(D23-K) -> /Vcc
- D71 pad 1: Net-(D23-K) -> /Vcc
- D72 pad 1: Net-(D23-K) -> /Vcc
- D73 pad 1: Net-(D23-K) -> /Vcc
- D74 pad 1: Net-(D23-K) -> /Vcc
- D75 pad 1: Net-(D23-K) -> /Vcc
- D76 pad 1: Net-(D23-K) -> /Vcc
- D77 pad 1: Net-(D23-K) -> /Vcc
- D78 pad 1: Net-(D23-K) -> /Vcc
- D79 pad 1: Net-(D23-K) -> /Vcc
- D80 pad 1: Net-(D23-K) -> /Vcc
- D81 pad 1: Net-(D23-K) -> /Vcc
- D82 pad 1: Net-(D23-K) -> /Vcc
- D83 pad 1: Net-(D23-K) -> /Vcc
- D84 pad 1: Net-(D23-K) -> /Vcc
- D85 pad 1: Net-(D100-K) -> /Vcc
- D86 pad 1: Net-(D100-K) -> /Vcc
- D87 pad 1: Net-(D100-K) -> /Vcc
- D88 pad 1: Net-(D100-K) -> /Vcc
- D89 pad 1: Net-(D100-K) -> /Vcc
- D90 pad 1: Net-(D100-K) -> /Vcc
- D91 pad 1: Net-(D100-K) -> /Vcc
- D92 pad 1: Net-(D100-K) -> /Vcc
- D93 pad 1: Net-(D100-K) -> /Vcc
- D94 pad 1: Net-(D100-K) -> /Vcc
- D95 pad 1: Net-(D100-K) -> /Vcc
- D96 pad 1: Net-(D100-K) -> /Vcc
- D97 pad 1: Net-(D100-K) -> /Vcc
- D98 pad 1: Net-(D100-K) -> /Vcc
- D99 pad 1: Net-(D100-K) -> /Vcc
- Q10 pad 1: Net-(D33-K) -> /Vcc
- Q11 pad 1: Net-(D117-K) -> /Vcc
- Q8 pad 1: Net-(D100-K) -> /Vcc
- Q9 pad 1: Net-(D23-K) -> /Vcc
- R1 pad 1: Net-(U1-VO) -> /Vcc
- R10 pad 1: /Vcc -> /digit 1
- R10 pad 2: Net-(D100-K) -> /Vcc
- R2 pad 1: /MCU/Vcc -> /Vcc
- R2 pad 2: Net-(U3-32KHZ) -> /MCU/32khz
- R21 pad 1: /Vcc -> /digit 2
- R21 pad 2: Net-(D23-K) -> /Vcc
- R22 pad 1: /Vcc -> /digit 1
- R23 pad 1: /Vcc -> /digit 2
- R24 pad 1: /Vcc -> /digit 3
- R24 pad 2: Net-(D33-K) -> Net-(Q10-B)
- R25 pad 2: Net-(Q10-B) -> /digit 3
- R26 pad 1: /Vcc -> /digit 4
- R26 pad 2: Net-(D117-K) -> /Vcc
- R27 pad 1: /Vcc -> /digit 4
- R3 pad 1: /MCU/Vcc -> /SQW
- R3 pad 2: Net-(U3-~{INT}/SQW) -> /Vcc
- R4 pad 1: /MCU/Vcc -> /Vcc
- R4 pad 2: /MCU/SCL -> /Vcc
- R5 pad 1: /MCU/Vcc -> /Vcc
- R5 pad 2: /MCU/SDA -> /Vcc
- U1 pad 3: Net-(U1-VO) -> /Vcc
- U2 pad 1: /MCU/RST -> unconnected-(U2-~{RESET}/PC6-Pad1)
- U2 pad 11: /MCU/Led D -> /Led D
- U2 pad 12: /MCU/Led E -> /Led E
- U2 pad 13: unconnected-(U2-PD7-Pad13) -> /Led G
- U2 pad 14: /MCU/Led G -> /Led F
- U2 pad 15: unconnected-(U2-PB1-Pad15) -> /digit 4
- U2 pad 16: unconnected-(U2-PB2-Pad16) -> /digit 3
- U2 pad 17: unconnected-(U2-PB3-Pad17) -> /digit 2
- U2 pad 18: unconnected-(U2-PB4-Pad18) -> /digit 1
- U2 pad 27: /MCU/SDA -> /Vcc
- U2 pad 28: /MCU/SCL -> /Vcc
- U2 pad 4: /MCU/Led A -> /Led A
- U2 pad 5: /MCU/Led B -> /Led B
- U2 pad 6: /MCU/Led C -> /Led C
- U2 pad 7: /MCU/Vcc -> /Vcc
- U3 pad 1: Net-(U3-32KHZ) -> unconnected-(U3-32KHZ-Pad1)
- U3 pad 10: GND -> Net-(U3-GND-Pad10)
- U3 pad 11: GND -> Net-(U3-GND-Pad10)
- U3 pad 12: GND -> Net-(U3-GND-Pad10)
- U3 pad 13: GND -> Net-(U3-GND-Pad10)
- U3 pad 15: /MCU/SDA -> unconnected-(U3-SDA-Pad15)
- U3 pad 16: /MCU/SCL -> unconnected-(U3-SCL-Pad16)
- U3 pad 2: /MCU/Vcc -> unconnected-(U3-VCC-Pad2)
- U3 pad 3: Net-(U3-~{INT}/SQW) -> unconnected-(U3-~{INT}/SQW-Pad3)
- U3 pad 4: /MCU/RST -> unconnected-(U3-~{RST}-Pad4)
- U3 pad 5: GND -> Net-(U3-GND-Pad10)
- U3 pad 6: GND -> Net-(U3-GND-Pad10)
- U3 pad 7: GND -> Net-(U3-GND-Pad10)
- U3 pad 8: GND -> Net-(U3-GND-Pad10)
- U3 pad 9: GND -> Net-(U3-GND-Pad10)
Routing:
- net /Vcc: track 0.00 -> 1447.1 mm, vias 0 -> 14
- net /E: track 0.00 -> 361.5 mm, vias 0 -> 4
- net /F: track 0.00 -> 349.0 mm, vias 0 -> 5
- net /C: track 0.00 -> 310.7 mm, vias 0 -> 4
- net /B: track 0.00 -> 287.0 mm, vias 0 -> 4
- net /A: track 0.00 -> 272.0 mm
- net /D: track 0.00 -> 269.5 mm
- net /G: track 0.00 -> 256.1 mm
- net /digit 1: track 0.00 -> 236.2 mm
- net /digit 2: track 0.00 -> 196.1 mm
- net /Led A: track 0.00 -> 160.9 mm
- net /SQW: track 0.00 -> 153.1 mm, vias 0 -> 2
- net /Led B: track 0.00 -> 138.3 mm
- net /Led F: track 0.00 -> 115.7 mm
- net /digit 3: track 0.00 -> 112.0 mm
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- added copper zone on B.Cu, net /Vcc
- removed copper zone on B.Cu, net (none)
Other:
- board size 214 x 150 mm -> 379.7 x 252 mm

Commit message: Vcc plane
Routing:
- net /B: track 287.0 -> 311.0 mm
- added copper zone on F.Cu, net /Vcc
- added copper zone on B.Cu, net GND
- removed copper zone on B.Cu, net /Vcc
Changed lines of the file:
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@@
 		(tags "Resistor Axial_DIN0207 series Axial Horizontal pin pitch 10.16mm 0.25W = 1/4W length 6.3mm diameter 2.5mm")
 		(property "Reference" "R37"
-			(at 5.08 -2.37 360)
+			(at 5.08 -2.37 0)
 			(layer "F.SilkS")
 			(effects
@@
 		)
 		(property "Value" "33"
-			(at 5.08 2.37 360)
+			(at 5.08 2.37 0)
 			(layer "F.Fab")
 			(effects
@@
 		)
 		(fp_text user "${REFERENCE}"
-			(at 4.84 0 360)
+			(at 4.84 0 0)
 			(layer "F.Fab")
 			(effects
@@
 		(tags "connector Molex SL vertical")
 		(property "Reference" "J1"
-			(at 16.51 -3.75 360)
+			(at 16.51 -3.75 0)
 			(layer "F.SilkS")
 			(effects
@@
 		)
 		(property "Value" "Conn_01x14_Socket"
-			(at 16.51 5.25 360)
+			(at 16.51 5.25 0)
 			(layer "F.Fab")
 			(effects
@@
 		)
 		(fp_text user "${REFERENCE}"
-			(at 16.51 1.85 360)
+			(at 16.51 1.85 0)
 			(layer "F.Fab")
 			(effects
@@
 		)
 		(fp_text user "${REFERENCE}"
-			(at 0 6.35 360)
+			(at 0 6.35 0)
 			(layer "F.Fab")
 			(effects
@@
 		(tags "Resistor Axial_DIN0207 series Axial Horizontal pin pitch 10.16mm 0.25W = 1/4W length 6.3mm diameter 2.5mm")
 		(property "Reference" "R36"
-			(at 5.08 -2.37 360)
+			(at 5.08 -2.37 0)
 			(layer "F.SilkS")
 			(effects
@@
 		)
 		(property "Value" "1k"
-			(at 5.08 2.37 360)
+			(at 5.08 2.37 0)
 			(layer "F.Fab")
 			(effects
@@
 		)
 		(fp_text user "${REFERENCE}"
-			(at 5.08 0 360)
+			(at 5.08 0 0)
 			(layer "F.Fab")
 			(effects
@@
 	)
 	(segment
-		(start 166 56.5)
-		(end 166.5 56)
+		(start 217 56)
+		(end 258 56)
 		(width 1)
 		(layer "F.Cu")
@@
 	)
 	(segment
-		(start 217 56)
-		(end 258 56)
+		(start 166 56.5)
+		(end 166.5 56)
 		(width 1)
 		(layer "F.Cu")
@@
 	)
 	(segment
+		(start 203.275 36)
+		(end 203.275 59.99)
+		(width 1)
+		(layer "B.Cu")
+		(net 38)
+	)
+	(segment
+		(start 203.275 59.99)
+		(end 203.265 60)
+		(width 1)
+		(layer "B.Cu")
+		(net 38)
+	)
+	(segment
 		(start 253.5 36)
 		(end 257 39.5)
@@
 		(net 3)
 		(net_name "/Vcc")
+		(layer "F.Cu")
+		(hatch edge 0.5)
+		(priority 1)
+		(connect_pads
+			(clearance 0.5)
+		)
+		(min_thickness 0.25)
+		(filled_areas_thickness no)
+		(fill yes
+			(thermal_gap 0.5)
+			(thermal_bridge_width 0.5)
+			(island_removal_mode 1)
+			(island_area_min 10)
+		)
+		(polygon
+			(pts
+				(xy 22.5 16) (xy 317 16.5) (xy 317 163.5) (xy 23.5 164)
+			)
+		)
+	)
+	(zone
+		(net 1)
+		(net_name "GND")
 		(layer "B.Cu")
 		(hatch edge 0.5)
@@
 		(polygon
 			(pts
-				(xy 24.5 18.5) (xy 315 18.5) (xy 315 162.5) (xy 25.5 163)
+				(xy 22.5 16) (xy 317 16) (xy 317.5 163) (xy 23.5 164)
 			)
 		)
